File: esp32 caliper.kicad_sch (KiCad schematic)
At the start: 44 parts, among them J1 USB4105-GF-A, J2 Current Testing, Q1 BC846BLT1G, Q2 BC846BLT1G, Q3 SSM3K36FS, SW1 Boot, SW2 Rst, SW3 SendEnter, SW4 SendSpace, U1 MCP73831T-5ACI/OT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

Commit message: add 1.5v output
Parts:
- added C6, C7: 1u, Capacitor_SMD:C_0402_1005Metric, symbol Device:C
- added U5: LP5907MFX-1.5/NOPB, SOT95P280X145-5N, symbol 1V5Reg:LP5907MFX-1.5/NOPB
Connections:
- net CLKIN: now also U2.2 (CLK); no longer U2.1 (CLK)
- net DATAIN: now also U2.3 (DATA); no longer U2.2 (DATA)
- net GND: now also U2.4 (GND), C6.2, C7.2, U5.2 (GND); no longer U2.3 (GND)
- net VDD: now also C6.1, U5.1 (IN), U5.3 (EN)
- new net +1V5: C7.1, U2.1 (1V5), U5.5 (OUT)
